Commit message: added world

File: mid-semester-exams-practicals-robottt/src/rover_description/urdf/rover.urdf.xacro (robot description, xacro)
@@ -5,5 +5,5 @@
     <color rgba="0.615686 0.811765 0.929412 1"/>
   </material>
-  <!-- body -->
+  <!-- Robot body -->
   <link name="base_link"/>
   <link name="main_body">
@@ -33,5 +33,5 @@
     <child link="main_body"/>
   </joint>
-  <!-- reusable wheel -->
+  <!-- Wheel macro -->
   <xacro:macro name="wheel" params="name xyz rpy axis inertial_xyz visual_xyz">
     <link name="${name}">
@@ -69,5 +69,5 @@
     </gazebo>
   </xacro:macro>
-  <!-- left-front: based on Planar 1 branch -->
+  <!-- Wheels  -->
   <xacro:wheel
       name="wheel_2"
@@ -77,5 +77,4 @@
       inertial_xyz="0.0143801 0 -0.00317342"
       visual_xyz="0.001 0 0"/>
-  <!-- right-front: based on Planar 2 branch -->
   <xacro:wheel
       name="wheel_1"
@@ -85,5 +84,4 @@
       inertial_xyz="0.0143801 0 -0.00317342"
       visual_xyz="0.001 0 0"/>
-  <!-- right-rear: based on Planar 3 branch -->
   <xacro:wheel
       name="wheel"
@@ -93,5 +91,4 @@
       inertial_xyz="0.0133801 0 -0.00317342"
       visual_xyz="0 0 0"/>
-  <!-- left-rear: based on Planar 4 branch -->
   <xacro:wheel
       name="wheel_3"
@@ -101,3 +98,131 @@
       inertial_xyz="0.0133801 0 -0.00317342"
       visual_xyz="0 0 0"/>
+  <!-- Lidar sensor link -->
+  <link name="lidar_link">
+    <inertial>
+      <mass value="0.1"/>
+      <inertia ixx="0.00007" ixy="0.0" ixz="0.0"
+               iyy="0.00007" iyz="0.0"
+               izz="0.00006"/>
+    </inertial>
+    <visual>
+      <geometry>
+        <cylinder radius="0.04" length="0.04"/>
+      </geometry>
+      <material name="body_color"/>
+    </visual>
+    <collision>
+      <geometry>
+        <cylinder radius="0.04" length="0.04"/>
+      </geometry>
+    </collision>
+  </link>
+  <joint name="lidar_joint" type="fixed">
+    <parent link="main_body"/>
+    <child link="lidar_link"/>
+    <origin xyz="-0.08 0.0 0.02" rpy="0 0 0"/>
+  </joint>
+  <!-- Camera link -->
+  <!-- Front facing camera for gem detection -->
+  <link name="camera_link">
+    <inertial>
+      <mass value="0.05"/>
+      <inertia ixx="0.00002" ixy="0.0" ixz="0.0"
+               iyy="0.00002" iyz="0.0"
+               izz="0.00002"/>
+    </inertial>
+    <visual>
+      <geometry>
+        <box size="0.025 0.025 0.025"/>
+      </geometry>
+      <material name="body_color"/>
+    </visual>
+    <collision>
+      <geometry>
+        <box size="0.025 0.025 0.025"/>
+      </geometry>
+    </collision>
+  </link>
+  <joint name="camera_joint" type="fixed">
+    <parent link="main_body"/>
+    <child link="camera_link"/>
+    <origin xyz="-0.04 0.0 0.01" rpy="0 0 0"/>
+  </joint>
+  <!-- gazebo plugins -->
+  <!-- Differential drive plugin -->
+  <!-- Allows the robot to move by subscribing to /cmd_vel -->
+  <gazebo>
+    <plugin filename="gz-sim-diff-drive-system"
+            name="gz::sim::systems::DiffDrive">
+      <left_joint>wheel_2_joint</left_joint>
+      <left_joint>wheel_3_joint</left_joint>
+      <right_joint>wheel_1_joint</right_joint>
+      <right_joint>wheel_joint</right_joint>
+      <wheel_separation>0.22</wheel_separation>
+      <wheel_radius>0.04</wheel_radius>
+      <max_linear_velocity>0.5</max_linear_velocity>
+      <max_angular_velocity>1.0</max_angular_velocity>
+      <max_linear_acceleration>1.0</max_linear_acceleration>
+      <topic>cmd_vel</topic>
+      <odom_topic>odom</odom_topic>
+      <frame_id>odom</frame_id>
+      <child_frame_id>base_link</child_frame_id>
+    </plugin>
+  </gazebo>
+  <!-- Joint state publisher plugin -->
+  <!-- Publishes the state of all joints -->
+  <gazebo>
+    <plugin filename="gz-sim-joint-state-publisher-system"
+            name="gz::sim::systems::JointStatePublisher">
+    </plugin>
+  </gazebo>
+  <!-- LIDAR sensor plugin -->
+  <!-- Gives the robot 360 degree wall detection -->
+  <gazebo reference="lidar_link">
+    <sensor name="lidar" type="gpu_lidar">
+      <always_on>true</always_on>
+      <visualize>true</visualize>
+      <update_rate>10</update_rate>
+      <topic>scan</topic>
+      <gz_frame_id>lidar_link</gz_frame_id>
+      <lidar>
+        <scan>
+          <horizontal>
+            <samples>360</samples>
+            <resolution>1</resolution>
+            <min_angle>-3.14159</min_angle>
+            <max_angle>3.14159</max_angle>
+          </horizontal>
+        </scan>
+        <range>
+          <min>0.10</min>
+          <max>10.0</max>
+          <resolution>0.01</resolution>
+        </range>
+      </lidar>
+    </sensor>
+  </gazebo>
+  <!-- Camera sensor plugin -->
+  <!-- Front facing camera for gem colour detection -->
+  <gazebo reference="camera_link">
+    <sensor name="camera" type="camera">
+      <always_on>true</always_on>
+      <visualize>true</visualize>
+      <update_rate>30</update_rate>
+      <topic>camera/image_raw</topic>
+      <gz_frame_id>camera_link</gz_frame_id>
+      <camera>
+        <horizontal_fov>1.3962634</horizontal_fov>
+        <image>
+          <width>640</width>
+          <height>480</height>
+          <format>R8G8B8</format>
+        </image>
+        <clip>
+          <near>0.02</near>
+          <far>300</far>
+        </clip>
+      </camera>
+    </sensor>
+  </gazebo>
 </robot>

Commit message: error_1 mesh collision issues saved reslovle att1

File: mid-semester-exams-practicals-robottt/src/rover_description/urdf/rover.urdf.xacro (robot description, xacro)
@@ -22,7 +22,7 @@
     </visual>
     <collision>
-      <origin xyz="8.67362e-19 0.00232656 -0.028" rpy="0 0 0"/>
-      <geometry>
-        <mesh filename="${mesh_dir}/59.stl" scale="1 1 1"/>
+      <origin xyz="0 0 -0.028" rpy="0 0 0"/>
+      <geometry>
+        <box size="0.22 0.18 0.08"/>
       </geometry>
     </collision>
@@ -49,10 +49,10 @@
         <material name="body_color"/>
       </visual>
-      <collision>
-        <origin xyz="${visual_xyz}" rpy="0 0 0"/>
+       <collision>
+        <origin xyz="0 0 0" rpy="1.5708 0 0"/>
         <geometry>
-          <mesh filename="${mesh_dir}/63.stl" scale="1 1 1"/>
+          <cylinder radius="0.04" length="0.02"/>
         </geometry>
-      </collision>
+    </collision>
     </link>
     <joint name="${name}_joint" type="continuous">
